File: pi-xp/pi-xp.sch (KiCad schematic (older format))
At the start: 21 parts

Commit message: pi_xp v1.1
Parts:
- removed OUT1, OUT2, OUT3: CONN_01X03, Pin_Headers:Pin_Header_Straight_1x03_Pitch2.54mm, symbol CONN_01X03
- added OUT1, OUT2, OUT3: CONN_01X02, Pin_Headers:Pin_Header_Straight_1x02_Pitch2.54mm, symbol CONN_01X02
- F1: footprint Fuse_Holders_and_Fuses:BladeFuse-Mini_Keystone_3568 -> Fuse_Holders_and_Fuses:Fuse_TE5_Littlefuse-395Series
Connections:
- net GND: now also OUT1.1 (P1), OUT2.1 (P1), OUT3.1 (P1)
- net OUTPUT1: now also OUT1.2 (P2)
- net OUTPUT2: now also OUT2.2 (P2)
- net OUTPUT3: now also OUT3.2 (P2)
Other:
- note added: "OyaMist Raspberry Pi GPIO extender"
- note added: "v1.1"
- note removed: "OyaMist Raspberry Pi GPIO power extender"
- note removed: "v1.0"
- moved on the sheet: FAN1
Changed lines of the file:
@@
 Text GLabel 7400 4100 0    60   Input ~ 0
 5V2
-$Comp
-L CONN_01X03 OUT1
-U 1 1 5AD14EA8
-P 3250 5200
-F 0 "OUT1" H 3250 5400 50  0000 C CNN
-F 1 "CONN_01X03" V 3350 5200 50  0001 C CNN
-F 2 "Pin_Headers:Pin_Header_Straight_1x03_Pitch2.54mm" H 3250 5200 50  0001 C CNN
-F 3 "" H 3250 5200 50  0000 C CNN
-	1    3250 5200
-	1    0    0    1
-$EndComp
 Text GLabel 3050 5300 0    60   Input ~ 0
 GND
-Text GLabel 3050 5100 0    60   Input ~ 0
-5V2
 Text GLabel 1250 2650 0    60   Output ~ 0
 OUTPUT3
@@
 Text GLabel 3050 5200 0    60   Input ~ 0
 OUTPUT1
-$Comp
-L CONN_01X03 OUT2
-U 1 1 5AD1570C
-P 4200 5200
-F 0 "OUT2" H 4200 5400 50  0000 C CNN
-F 1 "CONN_01X03" V 4300 5200 50  0001 C CNN
-F 2 "Pin_Headers:Pin_Header_Straight_1x03_Pitch2.54mm" H 4200 5200 50  0001 C CNN
-F 3 "" H 4200 5200 50  0000 C CNN
-	1    4200 5200
-	1    0    0    1
-$EndComp
 Text GLabel 4000 5300 0    60   Input ~ 0
 GND
-Text GLabel 4000 5100 0    60   Input ~ 0
-5V2
 Text GLabel 4000 5200 0    60   Input ~ 0
 OUTPUT2
-$Comp
-L CONN_01X03 OUT3
-U 1 1 5AD157A6
-P 5150 5200
-F 0 "OUT3" H 5150 5400 50  0000 C CNN
-F 1 "CONN_01X03" V 5250 5200 50  0001 C CNN
-F 2 "Pin_Headers:Pin_Header_Straight_1x03_Pitch2.54mm" H 5150 5200 50  0001 C CNN
-F 3 "" H 5150 5200 50  0000 C CNN
-	1    5150 5200
-	1    0    0    1
-$EndComp
 Text GLabel 4950 5300 0    60   Input ~ 0
 GND
-Text GLabel 4950 5100 0    60   Input ~ 0
-5V2
 Text GLabel 4950 5200 0    60   Input ~ 0
 OUTPUT3
@@
 L CONN_01X04 FAN1
 U 1 1 5AD174AD
-P 1550 6800
-F 0 "FAN1" H 1550 7050 50  0000 C CNN
-F 1 "CONN_01X04" V 4100 6750 50  0001 C CNN
-F 2 "Connect:Fan_Pin_Header_Straight_1x04" H 1450 7250 50  0001 C CNN
-F 3 "" H 1550 6800 50  0000 C CNN
-	1    1550 6800
-	1    0    0    1
-$EndComp
-Text GLabel 1350 6950 0    60   Input ~ 0
-GND
-Text GLabel 1350 6850 0    60   Input ~ 0
+P 1600 4550
+F 0 "FAN1" H 1600 4800 50  0000 C CNN
+F 1 "CONN_01X04" V 4150 4500 50  0001 C CNN
+F 2 "Connect:Fan_Pin_Header_Straight_1x04" H 1500 5000 50  0001 C CNN
+F 3 "" H 1600 4550 50  0000 C CNN
+	1    1600 4550
+	1    0    0    1
+$EndComp
+Text GLabel 1400 4700 0    60   Input ~ 0
+GND
+Text GLabel 1400 4600 0    60   Input ~ 0
 V12
-Text GLabel 1350 6650 0    60   Input ~ 0
+Text GLabel 1400 4400 0    60   Input ~ 0
 PWM
 $Comp
@@
 Text GLabel 7400 5150 0    60   Input ~ 0
 V12
-Text Notes 650  6300 0    79   ~ 0
+Text Notes 600  3750 0    79   ~ 0
 FAN\n\n
 Wire Notes Line
@@
 Text Notes 6750 800  0    79   ~ 0
 NO CONNECTION\n\n
-Text GLabel 1350 6750 0    60   Input ~ 0
+Text GLabel 1400 4500 0    60   Input ~ 0
 TACH
 Text GLabel 9050 1350 0    60   Input ~ 0
@@
 NoConn ~ 7700 2650
 NoConn ~ 7700 2750
-Text Notes 8700 6700 2    60   ~ 0
-OyaMist Raspberry Pi GPIO power extender
+Text Notes 9050 6750 2    60   ~ 0
+OyaMist Raspberry Pi GPIO extender
 Text Notes 10800 7650 2    60   ~ 0
-v1.0
+v1.1
 Text Notes 8700 7650 2    60   ~ 0
 2018-04-17
@@
 F 0 "F1" H 9550 4350 50  0000 C CNN
 F 1 "5A" H 9350 4250 50  0000 C CNN
-F 2 "Fuse_Holders_and_Fuses:BladeFuse-Mini_Keystone_3568" H 9450 4300 50  0001 C CNN
+F 2 "Fuse_Holders_and_Fuses:Fuse_TE5_Littlefuse-395Series" H 9450 4300 50  0001 C CNN
 F 3 "" H 9450 4300 50  0000 C CNN
 	1    9450 4300
@@
 Text GLabel 9100 4900 2    60   Input ~ 0
 GND
+$Comp
+L CONN_01X02 OUT1
+U 1 1 5AEA41D0
+P 3250 5250
+F 0 "OUT1" H 3250 5400 50  0000 C CNN
+F 1 "CONN_01X02" V 3350 5250 50  0001 C CNN
+F 2 "Pin_Headers:Pin_Header_Straight_1x02_Pitch2.54mm" H 3250 5250 50  0001 C CNN
+F 3 "" H 3250 5250 50  0000 C CNN
+	1    3250 5250
+	1    0    0    1
+$EndComp
+$Comp
+L CONN_01X02 OUT2
+U 1 1 5AEA4793
+P 4200 5250
+F 0 "OUT2" H 4200 5400 50  0000 C CNN
+F 1 "CONN_01X02" V 4300 5250 50  0001 C CNN
+F 2 "Pin_Headers:Pin_Header_Straight_1x02_Pitch2.54mm" H 4200 5250 50  0001 C CNN
+F 3 "" H 4200 5250 50  0000 C CNN
+	1    4200 5250
+	1    0    0    1
+$EndComp
+$Comp
+L CONN_01X02 OUT3
+U 1 1 5AEA4803
+P 5150 5250
+F 0 "OUT3" H 5150 5400 50  0000 C CNN
+F 1 "CONN_01X02" V 5250 5250 50  0001 C CNN
+F 2 "Pin_Headers:Pin_Header_Straight_1x02_Pitch2.54mm" H 5150 5250 50  0001 C CNN
+F 3 "" H 5150 5250 50  0000 C CNN
+	1    5150 5250
+	1    0    0    1
+$EndComp
 $EndSCHEMATC

Commit message: PI_XP1.2
Parts:
- removed OUT1, OUT2, OUT3: CONN_01X02, Pin_Headers:Pin_Header_Straight_1x02_Pitch2.54mm, symbol CONN_01X02
- added OUT1, OUT2, OUT3: CONN_01X03, Pin_Headers:Pin_Header_Straight_1x03_Pitch2.54mm, symbol CONN_01X03
Connections:
- net GND: now also OUT1.1 (P1), OUT2.1 (P1), OUT3.1 (P1)
- net OUTPUT1: now also OUT1.3 (P3)
- net OUTPUT2: now also OUT2.3 (P3)
- net OUTPUT3: now also OUT3.3 (P3)
- net PI3V3: now also OUT1.2 (P2), OUT2.2 (P2), OUT3.2 (P2)
Other:
- note added: "v1.2"
- note removed: "v1.1"
Changed lines of the file:
@@
 Text GLabel 1250 2350 0    60   BiDi ~ 0
 ID_SD
-Text GLabel 3050 5200 0    60   Input ~ 0
+Text GLabel 3050 5100 0    60   Input ~ 0
 OUTPUT1
 Text GLabel 4000 5300 0    60   Input ~ 0
 GND
-Text GLabel 4000 5200 0    60   Input ~ 0
+Text GLabel 4000 5100 0    60   Input ~ 0
 OUTPUT2
 Text GLabel 4950 5300 0    60   Input ~ 0
 GND
-Text GLabel 4950 5200 0    60   Input ~ 0
+Text GLabel 4950 5100 0    60   Input ~ 0
 OUTPUT3
 Text Notes 650  650  0    79   ~ 0
@@
 OyaMist Raspberry Pi GPIO extender
 Text Notes 10800 7650 2    60   ~ 0
-v1.1
+v1.2
 Text Notes 8700 7650 2    60   ~ 0
 2018-04-17
@@
 GND
 $Comp
-L CONN_01X02 OUT1
-U 1 1 5AEA41D0
-P 3250 5250
+L CONN_01X03 OUT1
+U 1 1 5AF20460
+P 3250 5200
 F 0 "OUT1" H 3250 5400 50  0000 C CNN
-F 1 "CONN_01X02" V 3350 5250 50  0001 C CNN
-F 2 "Pin_Headers:Pin_Header_Straight_1x02_Pitch2.54mm" H 3250 5250 50  0001 C CNN
-F 3 "" H 3250 5250 50  0000 C CNN
-	1    3250 5250
-	1    0    0    1
-$EndComp
-$Comp
-L CONN_01X02 OUT2
-U 1 1 5AEA4793
-P 4200 5250
+F 1 "CONN_01X03" V 3350 5200 50  0001 C CNN
+F 2 "Pin_Headers:Pin_Header_Straight_1x03_Pitch2.54mm" H 3250 5200 50  0001 C CNN
+F 3 "" H 3250 5200 50  0000 C CNN
+	1    3250 5200
+	1    0    0    1
+$EndComp
+$Comp
+L CONN_01X03 OUT2
+U 1 1 5AF206E7
+P 4200 5200
 F 0 "OUT2" H 4200 5400 50  0000 C CNN
-F 1 "CONN_01X02" V 4300 5250 50  0001 C CNN
-F 2 "Pin_Headers:Pin_Header_Straight_1x02_Pitch2.54mm" H 4200 5250 50  0001 C CNN
-F 3 "" H 4200 5250 50  0000 C CNN
-	1    4200 5250
-	1    0    0    1
-$EndComp
-$Comp
-L CONN_01X02 OUT3
-U 1 1 5AEA4803
-P 5150 5250
+F 1 "CONN_01X03" V 4300 5200 50  0001 C CNN
+F 2 "Pin_Headers:Pin_Header_Straight_1x03_Pitch2.54mm" H 4200 5200 50  0001 C CNN
+F 3 "" H 4200 5200 50  0000 C CNN
+	1    4200 5200
+	1    0    0    1
+$EndComp
+$Comp
+L CONN_01X03 OUT3
+U 1 1 5AF20753
+P 5150 5200
 F 0 "OUT3" H 5150 5400 50  0000 C CNN
-F 1 "CONN_01X02" V 5250 5250 50  0001 C CNN
-F 2 "Pin_Headers:Pin_Header_Straight_1x02_Pitch2.54mm" H 5150 5250 50  0001 C CNN
-F 3 "" H 5150 5250 50  0000 C CNN
-	1    5150 5250
-	1    0    0    1
-$EndComp
+F 1 "CONN_01X03" V 5250 5200 50  0001 C CNN
+F 2 "Pin_Headers:Pin_Header_Straight_1x03_Pitch2.54mm" H 5150 5200 50  0001 C CNN
+F 3 "" H 5150 5200 50  0000 C CNN
+	1    5150 5200
+	1    0    0    1
+$EndComp
+Text GLabel 4950 5200 0    60   Input ~ 0
+PI3V3
+Text GLabel 4000 5200 0    60   Input ~ 0
+PI3V3
+Text GLabel 3050 5200 0    60   Input ~ 0
+PI3V3
 $EndSCHEMATC

Commit message: v1.3
Other:
- note added: "NEOPIXEL\n\n\n"
- note added: "v1.3"
- note removed: "v1.2"
Changed lines of the file:
@@
 OyaMist Raspberry Pi GPIO extender
 Text Notes 10800 7650 2    60   ~ 0
-v1.2
+v1.3
 Text Notes 8700 7650 2    60   ~ 0
 2018-04-17
@@
 Text GLabel 3050 5200 0    60   Input ~ 0
 PI3V3
+Text Notes 600  6350 0    79   ~ 0
+NEOPIXEL\n\n\n
 $EndSCHEMATC

Commit message: v1.3
Other:
- note added: "2018-05-20"
- note removed: "2018-04-17"
Changed lines of the file:
@@
 v1.3
 Text Notes 8700 7650 2    60   ~ 0
-2018-04-17
+2018-05-20
 Text GLabel 1250 1050 0    60   Output ~ 0
 PI3V3_LED

Commit message: v1.4 I2C 3v3
Connections:
- net 5V2: no longer I2C1.2 (P2), I2C2.2 (P2), I2C3.2 (P2)
- net PI3V3_LED: now also I2C1.2 (P2), I2C2.2 (P2), I2C3.2 (P2)
Other:
- note added: "v1.4"
- note removed: "v1.3"
Changed lines of the file:
@@
 	1    0    0    -1
 $EndComp
-Text GLabel 3000 1200 0    60   Input ~ 0
-5V2
 Text GLabel 1750 1050 2    60   Input ~ 0
 5V2
@@
 	1    0    0    1
 $EndComp
-Text GLabel 4050 1200 0    60   Input ~ 0
-5V2
 Text GLabel 4050 1000 0    60   Input ~ 0
 I2C_CLK
@@
 	1    0    0    1
 $EndComp
-Text GLabel 5100 1200 0    60   Input ~ 0
-5V2
 Text GLabel 5100 1000 0    60   Input ~ 0
 I2C_CLK
@@
 OyaMist Raspberry Pi GPIO extender
 Text Notes 10800 7650 2    60   ~ 0
-v1.3
+v1.4
 Text Notes 8700 7650 2    60   ~ 0
 2018-05-20
@@
 Text Notes 600  6350 0    79   ~ 0
 NEOPIXEL\n\n\n
+Text GLabel 3000 1200 0    60   Input ~ 0
+PI3V3_LED
+Text GLabel 4050 1200 0    60   Input ~ 0
+PI3V3_LED
+Text GLabel 5100 1200 0    60   Input ~ 0
+PI3V3_LED
 $EndSCHEMATC
